File: VineHoop_V1_2.sch (KiCad schematic (older format))
At the start: 31 parts, among them J1 Conn_01x06_Female, J2 Conn_01x06_Female, J3 Conn_01x04_Female, U1 MIC5205-3.3YM5, U2 SHT31-DIS-B, U3 BNO055, U4 ATMEGA328P-MUR, Y1 32.768kHz, Y2 16MHz

Commit message: So much stuff
Parts:
- removed J1, J2: Conn_01x06_Female, Connector_PinHeader_2.54mm:PinHeader_1x06_P2.54mm_Vertical_SMD_Pin1Right, symbol Connector:Conn_01x06_Female
- removed J3: Conn_01x04_Female, Connector_PinHeader_2.54mm:PinHeader_1x04_P2.54mm_Vertical_SMD_Pin1Right, symbol Connector:Conn_01x04_Female
- removed Y1: 32.768kHz, XTAL_FC-135R_32.7680KA-AG0:XTAL_FC-135R_32.7680KA-AG0, symbol Device:Crystal
- removed Y2: 16MHz, 7A-16.000MAAE-T:XTAL_7A-16.000MAAE-T, symbol 7A-16.000MAAE-T:7A-16.000MAAE-T
- added J1: 95278-101A04LF, 4pin:95278101A04LF, symbol 95278-101A04LF:95278-101A04LF
- added J2, J3: 20021121-00006C4LF, 6pin:Amphenol_ICC___FCI-20021121-00006C4LF-MFG, symbol 6pin:20021121-00006C4LF
- added Y1: ABS07-32.768KHZ-T, ABS07-32.768KHZ-T:XTAL_ABS07-32.768KHZ-T, symbol ABS07-32.768KHZ-T:ABS07-32.768KHZ-T
- added Y2: ABM10-16.000MHZ-E20-T, ABM10-16.000MHZ-E20-T:XTAL250X200X50, symbol ABM10-16.000MHZ-E20-T:ABM10-16.000MHZ-E20-T
- renumbered C9 to C6, C6 to C7, C7 to C8, C8 to C9, D2 to D1, D1 to D2, R9 to R10, R10 to R11, R11 to R9
Connections:
- net +3V3: now also J3.4
- net GND: now also J1.1, J2.6, J3.6, Y2.2, Y2.4
- net MISO: now also J3.2
- net MOSI: now also J3.3
- net RESET: now also J3.5
- net RX: now also J2.2
- net SCK: now also J3.1
- net SCL: now also J1.2
- net SDA: now also J1.3
- net TX: now also J2.3
- net VDD: now also J1.4, J2.4
- net at C8.2, U4.7 (PB6): now also Y2.1 (XTAL@1)
- net at C9.2, U4.8 (PB7): now also Y2.3 (XTAL@2)
- net at C2.1, U3.26 (XOUT32): now also Y1.2
- net at C1.1, U3.27 (XIN32): now also Y1.1
