File: VineHoop_V1_2.kicad_pcb (KiCad board)
At the start: 2 copper layers, 49.3 x 15.2 mm, 31 parts, among them J1 95278-101A04LF, J2 20021121-00006C4LF, J3 20021121-00006C4LF, U1 MIC5205-3.3YM5, U2 SHT31-DIS-B, U3 BNO055, U4 ATMEGA328P-MUR, Y1 ABS07-32.768KHZ-T, Y2 ABM10-16.000MHZ-E20-T

Commit message: Lots of changes incl. "final" gerbers for rigid order
Other:
- net class Default removed
- net class Power removed
