File: VineHoop_Islands.kicad_sch (KiCad schematic)
At the start: 30 parts, among them J1 95278-101A04LF, J2 20021121-00006C4LF, U1 MIC5205-3.3YM5, U2 SHT31-DIS-B, U3 BNO055, U4 ATMEGA328P-MUR, Y1 ABS07-32.768KHZ-T, Y2 ABM10-16.000MHZ-E20-T

Commit message: First rough draft of islands
Connections:
- net SCL: now also J1.3; no longer J1.2
- net SDA: now also J1.2; no longer J1.3
Changed lines of the file:
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@@
     (effects (font (size 1.27 1.27)) (justify right))
   )
-  (global_label "SCL" (shape input) (at 127 111.76 180)
+  (global_label "SDA" (shape input) (at 127 111.76 180)
     (effects (font (size 1.27 1.27)) (justify right))
   )
-  (global_label "SDA" (shape input) (at 147.32 114.3 0)
+  (global_label "SCL" (shape input) (at 147.32 114.3 0)
     (effects (font (size 1.27 1.27)) (justify left))
   )

Commit message: Big backup
Parts:
- removed Y2: ABM10-16.000MHZ-E20-T, ABM10-16.000MHZ-E20-T:XTAL250X200X50, symbol ABM10-16.000MHZ-E20-T:ABM10-16.000MHZ-E20-T
- added R12, R13, R14, R15: 10K, Resistor_SMD:R_0603_1608Metric, symbol Device:R_Small
- added TH1, TH2, TH3, TH4: 10K, Resistor_SMD:R_0603_1608Metric, symbol Device:Thermistor_NTC
- C8: value 22pF -> 0.1uF
- C9: value 22pF -> 10uF
- U2: footprint SHT31-DIS-B:SON50P250X250X100-9N -> SHT31-V2:XDCR_SHT31-DIS-F2.5KS
Connections:
- net +3V3: now also C8.2, C9.1, TH1.1, TH2.1, TH3.1, TH4.1
- net GND: now also C9.2, R12.1, R13.1, R14.1, R15.1; no longer C9.1
- net MISO: now also J2.4; no longer J2.6
- net MOSI: now also J2.2; no longer J2.4
- net SCK: now also J2.6; no longer J2.2
- net SCL: now also J1.4; no longer J1.3
- net VDD: now also J1.3; no longer J1.4
- net A0: now reaches U4.23 (PC0)
- net A0: now also R12.2, TH1.2
- net A1: now reaches U4.24 (PC1)
- net A1: now also R13.2, TH2.2
- net A3: now reaches U4.26 (PC3)
- net A3: now also R15.2, TH4.2
- net at U4.7 (PB6): no longer C8.2
- net at U4.8 (PB7): no longer C9.2
- net PC2 renamed A2
- net A2: now also R14.2, TH3.2
